File: f1c200s.kicad_sch (KiCad schematic)
At the start: 44 parts, among them J1 Micro_SD_Card, J10 Conn_01x07, J2 USB_B_Micro, J3 Conn_01x03, J4 Conn_01x07, J5 Jumper, J6 Jumper, J7 Jumper, J8 Jumper, J9 Conn_01x01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

Commit message: Dev board V2
Parts:
- added J11: Conn_02x05_Odd_Even, Connector_PinHeader_2.54mm:PinHeader_2x05_P2.54mm_Vertical, symbol Connector_Generic:Conn_02x05_Odd_Even
- added J12: Conn_02x03_Odd_Even, Connector_PinHeader_2.54mm:PinHeader_2x03_P2.54mm_Vertical, symbol Connector_Generic:Conn_02x03_Odd_Even
- C1, C3, C5, C6: footprint Capacitor_SMD:C_0603_1608Metric -> Capacitor_SMD:C_0402_1005Metric; LCSC C19702 -> C15525
- C10, C11, C12, C13, C2, C4, C7, C8, C9: footprint Capacitor_SMD:C_0603_1608Metric -> Capacitor_SMD:C_0402_1005Metric; LCSC C15849 -> C52923
- J2: LCSC C132562 -> C132562
- Q1: LCSC C8545 -> C8545
- R1, R2: value 5.1K -> 4.7k; footprint Resistor_SMD:R_0603_1608Metric -> Resistor_SMD:R_0402_1005Metric; LCSC C23186 -> C25900
Connections:
- net GND: now also J11.1 (Pin_1), J11.8 (Pin_8), J12.5 (Pin_5)
- net I2C1_SCK: now also J11.6 (Pin_6)
- net I2C1_SDA: now also J11.5 (Pin_5)
- net PD0: now also J11.2 (Pin_2)
- net PD12: now also J11.7 (Pin_7)
- net PD13: now also J11.10 (Pin_10)
- net PD14: now also J11.9 (Pin_9)
- net PE6: now also J12.6 (Pin_6)
- net SPI1_CLK: now also J12.1 (Pin_1)
- net SPI1_CS: now also J12.3 (Pin_3)
- net SPI1_MISO: now also J12.2 (Pin_2)
- net SPI1_MOSI: now also J12.4 (Pin_4)
- net UART1_RX: now also J11.4 (Pin_4)
- net UART1_TX: now also J11.3 (Pin_3)
Other:
- moved on the sheet: J10, J3, J4
